File: cpu.kicad_sch (KiCad schematic)
At the start: 15 parts

Commit message: Fix wrong cap type in clock generator
Also fill some references automatically generated by KiCAD.
Parts:
- C15, C16, C17, C19, C3, C4: renamed from C?; value (none) -> 100nF; footprint (none) -> artemisa:Disc_capacitor
- U3, U4, U5: value (none) -> 74HCT244; footprint (none) -> artemisa:DIP-20_300
- U3, U4, U5: renamed from U?; value (none) -> 74HCT244; footprint (none) -> artemisa:DIP-20_300
- U6: value (none) -> Z84C00; footprint (none) -> artemisa:DIP-40_600
- U7: value (none) -> 74HC74; footprint (none) -> artemisa:DIP-14_300
- U8: value (none) -> 74HCT245; footprint (none) -> artemisa:DIP-20_300
Connections:
- net VCC: now reaches C3.1, U6.11 (VCC)
- net VCC: now also C15.1, C16.1, C17.1, C19.1, C4.1, U3.20 (VCC), U4.20 (VCC), U5.20 (VCC), U6.17 (~{NMI}), U6.25 (~{BUSREQ}), U7.13 (~{RD}), U7.14 (VCC), U8.20 (VCC)
