File: power.kicad_sch (KiCad schematic)
At the start: 18 parts

Commit message: Fix wrong cap type in clock generator
Also fill some references automatically generated by KiCAD.
Parts:
- C5: value (none) -> 100uF; footprint (none) -> artemisa:Radial_capacitor
- C6: value (none) -> 10uF; footprint (none) -> artemisa:Radial_capacitor
- C7: renamed from C?; value (none) -> 100uF; footprint (none) -> artemisa:Radial_capacitor
- C9: value (none) -> 100nF; footprint (none) -> artemisa:Disc_capacitor
- D1: value (none) -> 1N4448; footprint (none) -> artemisa:Axial_diode
- D2: value (none) -> LED; footprint (none) -> artemisa:LED
- J1: value (none) -> PWR_conn; footprint (none) -> artemisa:Jack_55_21
- Q1: value (none) -> 2N2222; footprint (none) -> artemisa:TO92
- R1: renamed from R?; value (none) -> 100K; footprint (none) -> artemisa:Axial_resistor
- R2: value (none) -> 220; footprint (none) -> artemisa:Axial_resistor
- R3, R6: renamed from R?; value (none) -> 4K7; footprint (none) -> artemisa:Axial_resistor
- R4: renamed from R?; value (none) -> 10K; footprint (none) -> artemisa:Axial_resistor
- R5: renamed from R?; value (none) -> 1K; footprint (none) -> artemisa:Axial_resistor
- SW1: value (none) -> Push_button; footprint (none) -> artemisa:Push_button_angled
- U9: renamed from U?; value (none) -> 74HCU04; footprint (none) -> artemisa:DIP-14_300
Connections:
- net RESET: now also U9.5; no longer U9.3
- net ~{RESET}: now also U9.6; no longer U9.4
- net VCC: now reaches C5.1, C6.1, J1.1 (VCC), R2.1
- net VCC: now also C9.1, D1.2, R3.1, R4.1, U9.14 (VCC)
