File: ppi.kicad_sch (KiCad schematic)
At the start: 6 parts

Commit message: Fix wrong cap type in clock generator
Also fill some references automatically generated by KiCAD.
Parts:
- C14, C39, C40: renamed from C?; value (none) -> 100nF; footprint (none) -> artemisa:Disc_capacitor
- U15: value (none) -> 74HC139; footprint (none) -> artemisa:DIP-16_300
- U27: value (none) -> 74HC153; footprint (none) -> artemisa:DIP-16_300
- U28: value (none) -> 82C55A; footprint (none) -> artemisa:DIP-40_600
Connections:
- net VCC: now reaches C40.1, U28.26 (VCC)
- net VCC: now also C14.1, C39.1, U15.16 (VCC), U27.16 (VCC)
Changed lines of the file:
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@@
       (effects (font (size 1.524 1.524)))
     )
-    (property "Value" "" (id 1) (at 121.92 160.02 0)
-      (effects (font (size 1.524 1.524)))
-    )
-    (property "Footprint" "" (id 2) (at 119.38 113.03 0)
+    (property "Value" "82C55A" (id 1) (at 121.92 160.02 0)
+      (effects (font (size 1.524 1.524)))
+    )
+    (property "Footprint" "artemisa:DIP-40_600" (id 2) (at 119.38 113.03 0)
       (effects (font (size 1.524 1.524)) hide)
     )
@@
       (effects (font (size 1.524 1.524)))
     )
-    (property "Value" "" (id 1) (at 167.64 78.74 0)
-      (effects (font (size 1.524 1.524)))
-    )
-    (property "Footprint" "" (id 2) (at 160.02 63.5 0)
+    (property "Value" "74HC153" (id 1) (at 167.64 78.74 0)
+      (effects (font (size 1.524 1.524)))
+    )
+    (property "Footprint" "artemisa:DIP-16_300" (id 2) (at 160.02 63.5 0)
       (effects (font (size 1.524 1.524)) hide)
     )
@@
       (effects (font (size 1.524 1.524)))
     )
-    (property "Value" "" (id 1) (at 215.9 60.96 0)
-      (effects (font (size 1.524 1.524)))
-    )
-    (property "Footprint" "" (id 2) (at 209.55 57.15 0)
+    (property "Value" "74HC139" (id 1) (at 215.9 60.96 0)
+      (effects (font (size 1.524 1.524)))
+    )
+    (property "Footprint" "artemisa:DIP-16_300" (id 2) (at 209.55 57.15 0)
       (effects (font (size 1.524 1.524)) hide)
     )
@@
       (effects (font (size 1.524 1.524)) hide)
     )
-    (property "Value" "" (id 1) (at 160.02 77.47 0)
+    (property "Value" "GND" (id 1) (at 160.02 77.47 0)
       (effects (font (size 1.524 1.524)) hide)
     )
@@
       (effects (font (size 1.524 1.524)) hide)
     )
-    (property "Value" "" (id 1) (at 160.02 27.94 0)
+    (property "Value" "VCC" (id 1) (at 160.02 27.94 0)
       (effects (font (size 1.524 1.524)) hide)
     )
@@
   (symbol (lib_id "artemisa:Cap") (at 168.91 35.56 90) (unit 1)
     (in_bom yes) (on_board yes)
-    (property "Reference" "C?" (id 0) (at 166.37 34.29 90)
+    (property "Reference" "C39" (id 0) (at 166.37 34.29 90)
       (effects (font (size 1.27 1.27)) (justify left))
     )
-    (property "Value" "" (id 1) (at 176.53 34.29 90)
+    (property "Value" "100nF" (id 1) (at 176.53 34.29 90)
       (effects (font (size 1.27 1.27)) (justify left))
     )
-    (property "Footprint" "" (id 2) (at 168.91 35.56 0)
+    (property "Footprint" "artemisa:Disc_capacitor" (id 2) (at 168.91 35.56 0)
       (effects (font (size 1.27 1.27)) hide)
     )
@@
       (effects (font (size 1.524 1.524)) hide)
     )
-    (property "Value" "" (id 1) (at 175.26 35.56 0)
+    (property "Value" "GND" (id 1) (at 175.26 35.56 0)
       (effects (font (size 1.524 1.524)) hide)
     )
@@
       (effects (font (size 1.524 1.524)) hide)
     )
-    (property "Value" "" (id 1) (at 93.98 154.94 0)
+    (property "Value" "GND" (id 1) (at 93.98 154.94 0)
       (effects (font (size 1.524 1.524)) hide)
     )
@@
       (effects (font (size 1.524 1.524)) hide)
     )
-    (property "Value" "" (id 1) (at 114.3 158.75 0)
+    (property "Value" "GND" (id 1) (at 114.3 158.75 0)
       (effects (font (size 1.524 1.524)) hide)
     )
@@
       (effects (font (size 1.524 1.524)) hide)
     )
-    (property "Value" "" (id 1) (at 114.3 73.66 0)
+    (property "Value" "VCC" (id 1) (at 114.3 73.66 0)
       (effects (font (size 1.524 1.524)) hide)
     )
@@
   (symbol (lib_id "artemisa:Cap") (at 121.92 83.82 90) (unit 1)
     (in_bom yes) (on_board yes)
-    (property "Reference" "C?" (id 0) (at 119.38 82.55 90)
+    (property "Reference" "C40" (id 0) (at 119.38 82.55 90)
       (effects (font (size 1.27 1.27)) (justify left))
     )
-    (property "Value" "" (id 1) (at 129.54 82.55 90)
+    (property "Value" "100nF" (id 1) (at 129.54 82.55 90)
       (effects (font (size 1.27 1.27)) (justify left))
     )
-    (property "Footprint" "" (id 2) (at 121.92 83.82 0)
+    (property "Footprint" "artemisa:Disc_capacitor" (id 2) (at 121.92 83.82 0)
       (effects (font (size 1.27 1.27)) hide)
     )
@@
       (effects (font (size 1.524 1.524)) hide)
     )
-    (property "Value" "" (id 1) (at 128.27 83.82 0)
+    (property "Value" "GND" (id 1) (at 128.27 83.82 0)
       (effects (font (size 1.524 1.524)) hide)
     )
@@
   (symbol (lib_id "artemisa:GND") (at 209.55 63.5 0) (unit 1)
     (in_bom yes) (on_board yes)
-    (property "Reference" "#PWR?" (id 0) (at 209.55 66.04 0)
-      (effects (font (size 1.524 1.524)) hide)
-    )
-    (property "Value" "" (id 1) (at 209.55 60.96 0)
+    (property "Reference" "#PWR0156" (id 0) (at 209.55 66.04 0)
+      (effects (font (size 1.524 1.524)) hide)
+    )
+    (property "Value" "GND" (id 1) (at 209.55 60.96 0)
       (effects (font (size 1.524 1.524)) hide)
     )
@@
   (symbol (lib_id "artemisa:VCC") (at 209.55 35.56 0) (unit 1)
     (in_bom yes) (on_board yes)
-    (property "Reference" "#PWR?" (id 0) (at 209.55 36.83 0)
-      (effects (font (size 1.524 1.524)) hide)
-    )
-    (property "Value" "" (id 1) (at 209.55 29.21 0)
+    (property "Reference" "#PWR0157" (id 0) (at 209.55 36.83 0)
+      (effects (font (size 1.524 1.524)) hide)
+    )
+    (property "Value" "VCC" (id 1) (at 209.55 29.21 0)
       (effects (font (size 1.524 1.524)) hide)
     )
@@
   (symbol (lib_id "artemisa:Cap") (at 218.44 38.1 90) (unit 1)
     (in_bom yes) (on_board yes)
-    (property "Reference" "C?" (id 0) (at 218.44 34.29 90))
-    (property "Value" "" (id 1) (at 218.44 41.91 90))
-    (property "Footprint" "" (id 2) (at 218.44 38.1 0)
+    (property "Reference" "C14" (id 0) (at 218.44 34.29 90))
+    (property "Value" "100nF" (id 1) (at 218.44 41.91 90))
+    (property "Footprint" "artemisa:Disc_capacitor" (id 2) (at 218.44 38.1 0)
       (effects (font (size 1.27 1.27)) hide)
     )
@@
   (symbol (lib_id "artemisa:GND") (at 226.06 41.91 0) (unit 1)
     (in_bom yes) (on_board yes)
-    (property "Reference" "#PWR?" (id 0) (at 226.06 44.45 0)
-      (effects (font (size 1.524 1.524)) hide)
-    )
-    (property "Value" "" (id 1) (at 226.06 39.37 0)
-      (effects (font (size 1.524 1.524)) hide)
-    )
+    (property "Reference" "#PWR0162" (id 0) (at 226.06 44.45 0)
+      (effects (font (size 1.524 1.524)) hide)
+    )
+    (property "Value" "GND" (id 1) (at 226.06 39.37 0)
+      (effects (font (size 1.524 1.524)) hide)
+    )
