File: psg.kicad_sch (KiCad schematic)
At the start: 21 parts

Commit message: Fix wrong cap type in clock generator
Also fill some references automatically generated by KiCAD.
Parts:
- C26, C27, C28: renamed from C?; value (none) -> 100nF; footprint (none) -> artemisa:Disc_capacitor
- C29, C30, C31: value (none) -> 10u; footprint (none) -> artemisa:Radial_capacitor
- J6, J7: value (none) -> CONN_JOY; footprint (none) -> artemisa:Joystick_conn
- R10: renamed from R?; value (none) -> 20k; footprint (none) -> artemisa:Axial_resistor
- R11: renamed from R?; value (none) -> 4k7; footprint (none) -> artemisa:Axial_resistor
- R12: renamed from R?; value (none) -> 2k7; footprint (none) -> artemisa:Axial_resistor
- R7, R9: renamed from R?; value (none) -> 10K; footprint (none) -> artemisa:Axial_resistor
- R8: renamed from R?; value (none) -> 470; footprint (none) -> artemisa:Axial_resistor
- RN4: value (none) -> 10K; footprint (none) -> artemisa:RN8
- RN5: value (none) -> 10K; footprint (none) -> artemisa:RN4
- U14: value (none) -> 74HC08; footprint (none) -> artemisa:DIP-14_300
- U16: value (none) -> 74LS07; footprint (none) -> artemisa:DIP-14_300
- U23, U25: value (none) -> 74HC157; footprint (none) -> artemisa:DIP-16_300
- U24: value (none) -> AY-3-8910; footprint (none) -> artemisa:DIP-40_600
Connections:
- net VCC: now also C26.1, C27.1, C28.1, J6.5 (VCC), J7.5 (VCC), R7.1, RN4.1, RN5.1, U23.16 (VCC), U24.25 (A8), U24.28 (BC2), U24.40 (VCC), U25.16 (VCC)
